File: Scanner1.kicad_pcb (KiCad board)
At the start: 2 copper layers, 99.1 x 50.2 mm, 45 parts, among them J1 0548190519, J2 Conn_02x05_Odd_Even, J3 Conn_02x03_Odd_Even, Q1 MOSFET_N, SW1 SW_Push, SW2 SW_Push, SW3 SW_Push, U1 ATmega32U4-AU, Y1 16 MHz X322516MLB4SI

Commit message: More layout
Parts:
- moved C2 74.1 mm to (186.1, 80.0), turned to 180 degrees
- moved Y1 66.4 mm to (186.1, 83.2), turned to 270 degrees
- moved C1 61.0 mm to (189.0, 83.2), turned to 270 degrees
- moved SW1 54.7 mm to (132.6, 88.4)
- moved R2 54.3 mm to (146.1, 91.1), turned to 270 degrees
- moved C8 51.8 mm to (163.4, 77.2), turned to 270 degrees
- moved R1 49.8 mm to (143.3, 91.1), turned to 270 degrees
- moved R7 47.6 mm to (198.8, 82.0)
- moved R8 47.6 mm to (212.2, 81.5)
- moved SW2 47.6 mm to (210.0, 87.9)
- moved SW3 47.6 mm to (199.5, 87.9)
- moved Q1 40.2 mm to (150.0, 70.9), turned to 180 degrees
- moved J2 39.9 mm to (158.0, 87.1), turned to 180 degrees
- moved R6 35.1 mm to (168.0, 72.6)
- moved C6 33.8 mm to (182.4, 85.2), turned to 90 degrees
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Routing:
- net RD+: track 0.00 -> 39.0 mm
- net RD-: track 0.00 -> 39.0 mm
- net Net-(D9-Pad2): track 0.00 -> 38.5 mm
- net Net-(D8-Pad2): track 0.00 -> 31.7 mm
- net LED_0: track 0.00 -> 28.1 mm
- net Net-(D7-Pad2): track 0.00 -> 24.9 mm
- net LED_1: track 0.00 -> 23.7 mm
- net Net-(D1-Pad2): track 0.00 -> 22.5 mm
- net LED_2: track 0.00 -> 19.7 mm
- net Net-(D6-Pad2): track 0.00 -> 18.5 mm
- net LED_3: track 0.00 -> 16.5 mm
- net MOSI: track 0.00 -> 16.1 mm
- net Net-(D2-Pad2): track 0.00 -> 16.1 mm
- net LED_4: track 0.00 -> 14.9 mm, vias 0 -> 2
- net GND: track 0.00 -> 14.8 mm, vias 0 -> 3
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- added copper zone on F.Cu, net GND
Other:
- board size 99.1 x 50.2 mm -> 99.1 x 40 mm

Commit message: Layout and routing complete. Still needs silkscreen work and optionally extra pieces to cover the light bar
Parts:
- moved SW3 19.6 mm to (219.1, 88.4)
- moved R7 17.9 mm to (215.1, 89.3), turned to 90 degrees
- moved J2 10.2 mm to (156.1, 77.1), turned to 0 degrees
- moved R8 7.78 mm to (212.9, 89.3), turned to 90 degrees
- moved SW2 7.75 mm to (202.3, 88.4)
- moved C8 0.96 mm to (164.0, 78.0)
- moved C5 0.68 mm to (164.0, 85.5)
- moved C7 0.62 mm to (172.3, 91.6)
- moved R6 0.27 mm to (168.2, 72.8)
Connections:
- U1 pad 30: SW_0 -> Net-(U1-Pad30)
- U1 pad 8: Net-(U1-Pad8) -> SW_0
Routing:
- net +5V: track 8.99 -> 158.8 mm, vias 0 -> 2
- net Net-(D1-Pad1): track 0.00 -> 144.9 mm
- net RST: track 9.84 -> 66.4 mm, vias 2 -> 4
- net SW_0: track 0.00 -> 39.8 mm
- net SW_1: track 14.2 -> 53.6 mm
- net TCK: track 0.00 -> 34.5 mm
- net LED_CTRL: track 2.43 -> 27.5 mm
- net GND: track 14.8 -> 36.3 mm, vias 3 -> 9
- net TDI: track 0.00 -> 16.5 mm, vias 0 -> 2
- net Net-(R1-Pad2): track 0.00 -> 15.0 mm
- net TMS: track 0.00 -> 12.8 mm
- net TDO: track 0.00 -> 12.0 mm
- net Net-(R6-Pad2): track 0.00 -> 3.73 mm
- net Net-(C7-Pad1): track 0.00 -> 3.70 mm
- net Net-(C5-Pad1): track 0.00 -> 3.59 mm
- added copper zone on B.Cu, net GND
